Commit message: Fix the issue with the serial port

File: mycobot_ros2/mycobot_description/urdf/mecharm_270_m5/mecharm_270_m5.urdf (robot description, URDF)
Before this commit: robot firefighter, 7 links, 6 joints
Joints:
- joint joint2_to_joint1: limit lower=-1.3089 upper=2.0943 effort=1000.0 velocity=0 -> lower=-1.48353 upper=1.570796 effort=1000.0 velocity=0
- joint joint3_to_joint2: limit lower=-3.0543 upper=1.1344 effort=1000.0 velocity=0 -> lower=-3.14 upper=0.785398 effort=1000.0 velocity=0
- joint joint4_to_joint3: limit lower=-2.7052 upper=2.7052 effort=1000.0 velocity=0 -> lower=-2.792527 upper=2.792527 effort=1000.0 velocity=0
- joint joint5_to_joint4: limit lower=-2.0071 upper=2.0071 effort=1000.0 velocity=0 -> lower=-1.745329 upper=1.745329 effort=1000.0 velocity=0

File: mycobot_ros2/mycobot_description/urdf/mecharm_270_pi/mecharm_270_pi.urdf (robot description, URDF)
Before this commit: robot firefighter, 7 links, 6 joints
Joints:
- joint joint2_to_joint1: limit lower=-1.3089 upper=2.0943 effort=1000.0 velocity=0 -> lower=-1.48353 upper=1.570796 effort=1000.0 velocity=0
- joint joint3_to_joint2: limit lower=-3.0543 upper=1.1344 effort=1000.0 velocity=0 -> lower=-3.14 upper=0.785398 effort=1000.0 velocity=0
- joint joint4_to_joint3: limit lower=-2.7052 upper=2.7052 effort=1000.0 velocity=0 -> lower=-2.792527 upper=2.792527 effort=1000.0 velocity=0
- joint joint5_to_joint4: limit lower=-2.0071 upper=2.0071 effort=1000.0 velocity=0 -> lower=-1.745329 upper=1.745329 effort=1000.0 velocity=0

File: mycobot_ros2/mycobot_description/urdf/myarm_300_pi/myarm_300_pi.urdf (robot description, URDF)
Before this commit: robot firefighter, 8 links, 7 joints
Joints:
- joint joint2_to_joint1: limit lower=-1.2217 upper=2.0071 effort=1000.0 velocity=0 -> lower=-1.3962 upper=1.3962 effort=1000.0 velocity=0
- joint joint3_to_joint2: limit lower=-2.9670 upper=2.9670 effort=1000.0 velocity=0 -> lower=-2.8797 upper=2.8797 effort=1000.0 velocity=0
- joint joint4_to_joint3: limit lower=-1.9722 upper=1.3089 effort=1000.0 velocity=0 -> lower=-1.7453 upper=1.3962 effort=1000.0 velocity=0
- joint joint5_to_joint4: limit lower=-2.9670 upper=2.9670 effort=1000.0 velocity=0 -> lower=-2.8797 upper=2.8797 effort=1000.0 velocity=0
- joint joint6_to_joint5: limit lower=-2.0071 upper=2.0071 effort=1000.0 velocity=0 -> lower=-1.9198 upper=1.9198 effort=1000.0 velocity=0
- joint joint7_to_joint6: limit lower=-3.14159 upper=3.14159 effort=1000.0 velocity=0 -> lower=-2.8797 upper=2.8797 effort=1000.0 velocity=0

File: mycobot_ros2/mycobot_description/urdf/mybuddy/mybuddy.urdf (robot description, URDF)
Before this commit: robot firefighter, 14 links, 13 joints
Joints:
- joint base_link1: limit lower=-2.0943 upper=2.0943 effort=1000.0 velocity=0 -> lower=-3.14 upper=3.14159 effort=1000.0 velocity=0
- joint joint1_L: limit lower=-2.8798 upper=2.8798 effort=1000.0 velocity=0 -> lower=-3.14 upper=3.14159 effort=1000.0 velocity=0
- joint joint1_R: limit lower=-2.8798 upper=2.8798 effort=1000.0 velocity=0 -> lower=-3.14 upper=3.14159 effort=1000.0 velocity=0
- joint joint2_L: limit lower=-2.8798 upper=2.8798 effort=1000.0 velocity=0 -> lower=-3.14 upper=3.14159 effort=1000.0 velocity=0
- joint joint2_R: limit lower=-2.8798 upper=2.8798 effort=1000.0 velocity=0 -> lower=-3.14 upper=3.14159 effort=1000.0 velocity=0
- joint joint3_L: limit lower=-2.8798 upper=2.8798 effort=1000.0 velocity=0 -> lower=-3.14 upper=3.14159 effort=1000.0 velocity=0
- joint joint3_R: limit lower=-2.8798 upper=2.8798 effort=1000.0 velocity=0 -> lower=-3.14 upper=3.14159 effort=1000.0 velocity=0
- joint joint4_L: limit lower=-2.8798 upper=2.8798 effort=1000.0 velocity=0 -> lower=-3.14 upper=3.14159 effort=1000.0 velocity=0
- joint joint4_R: limit lower=-2.8798 upper=2.8798 effort=1000.0 velocity=0 -> lower=-3.14 upper=3.14159 effort=1000.0 velocity=0
- joint joint5_L: limit lower=-2.8798 upper=2.8798 effort=1000.0 velocity=0 -> lower=-3.14 upper=3.14159 effort=1000.0 velocity=0
- joint joint5_R: limit lower=-2.8798 upper=2.8798 effort=1000.0 velocity=0 -> lower=-3.14 upper=3.14159 effort=1000.0 velocity=0
- joint joint6_L: limit lower=-3.0543 upper=3.0543 effort=1000.0 velocity=0 -> lower=-3.14 upper=3.14159 effort=1000.0 velocity=0
- joint joint6_R: limit lower=-3.0543 upper=3.0543 effort=1000.0 velocity=0 -> lower=-3.14 upper=3.14159 effort=1000.0 velocity=0

File: mycobot_ros2/mycobot_description/urdf/mycobot_280_jn/mycobot_280_jn.urdf (robot description, URDF)
Before this commit: robot firefighter, 7 links, 6 joints
Joints:
- joint joint2_to_joint1: limit lower=-2.9322 upper=2.9322 effort=1000.0 velocity=0 -> lower=-3.14 upper=3.14159 effort=1000.0 velocity=0
- joint joint3_to_joint2: limit lower=-2.3562 upper=2.3562 effort=1000.0 velocity=0 -> lower=-3.14 upper=3.14159 effort=1000.0 velocity=0
- joint joint4_to_joint3: limit lower=-2.618 upper=2.618 effort=1000.0 velocity=0 -> lower=-3.14 upper=3.14159 effort=1000.0 velocity=0
- joint joint5_to_joint4: limit lower=-2.5307 upper=2.5307 effort=1000.0 velocity=0 -> lower=-3.14 upper=3.14159 effort=1000.0 velocity=0
- joint joint6_to_joint5: limit lower=-2.8798 upper=2.8798 effort=1000.0 velocity=0 -> lower=-3.14 upper=3.14159 effort=1000.0 velocity=0
- joint joint6output_to_joint6: limit lower=-3.14159 upper=3.14159 effort=1000.0 velocity=0 -> lower=-3.14 upper=3.14159 effort=1000.0 velocity=0

File: mycobot_ros2/mycobot_description/urdf/mycobot_280_m5/mycobot_280_m5.urdf (robot description, URDF)
Before this commit: robot firefighter, 8 links, 7 joints
Joints:
- joint joint2_to_joint1: limit lower=-2.9322 upper=2.9322 effort=1000.0 velocity=0 -> lower=-3.14 upper=3.14159 effort=1000.0 velocity=0
- joint joint3_to_joint2: limit lower=-2.3562 upper=2.3562 effort=1000.0 velocity=0 -> lower=-3.14 upper=3.14159 effort=1000.0 velocity=0
- joint joint4_to_joint3: limit lower=-2.618 upper=2.618 effort=1000.0 velocity=0 -> lower=-3.14 upper=3.14159 effort=1000.0 velocity=0
- joint joint5_to_joint4: limit lower=-2.5307 upper=2.5307 effort=1000.0 velocity=0 -> lower=-3.14 upper=3.14159 effort=1000.0 velocity=0
- joint joint6_to_joint5: limit lower=-2.8798 upper=2.8798 effort=1000.0 velocity=0 -> lower=-3.14 upper=3.14159 effort=1000.0 velocity=0
- joint joint6output_to_joint6: limit lower=-3.14159 upper=3.14159 effort=1000.0 velocity=0 -> lower=-3.14 upper=3.14159 effort=1000.0 velocity=0

File: mycobot_ros2/mycobot_description/urdf/mycobot_280_m5/mycobot_280_m5_with_camera_flange.urdf (robot description, URDF)
Before this commit: robot firefighter, 9 links, 8 joints
Joints:
- joint joint2_to_joint1: limit lower=-2.9322 upper=2.9322 effort=1000.0 velocity=0 -> lower=-2.879793 upper=2.879793 effort=1000.0 velocity=0
- joint joint3_to_joint2: limit lower=-2.3562 upper=2.3562 effort=1000.0 velocity=0 -> lower=-2.879793 upper=2.879793 effort=1000.0 velocity=0
- joint joint4_to_joint3: limit lower=-2.618 upper=2.618 effort=1000.0 velocity=0 -> lower=-2.879793 upper=2.879793 effort=1000.0 velocity=0
- joint joint5_to_joint4: limit lower=-2.5307 upper=2.5307 effort=1000.0 velocity=0 -> lower=-2.879793 upper=2.879793 effort=1000.0 velocity=0
- joint joint6_to_joint5: limit lower=-2.8798 upper=2.8798 effort=1000.0 velocity=0 -> lower=-2.879793 upper=2.879793 effort=1000.0 velocity=0
- joint joint6output_to_joint6: limit lower=-3.14159 upper=3.14159 effort=1000.0 velocity=0 -> lower=-3.05 upper=3.05 effort=1000.0 velocity=0

File: mycobot_ros2/mycobot_description/urdf/mycobot_280_m5/mycobot_280_m5_with_camera_flange_pump.urdf (robot description, URDF)
Before this commit: robot firefighter, 11 links, 10 joints
Joints:
- joint joint2_to_joint1: limit lower=-2.9322 upper=2.9322 effort=1000.0 velocity=0 -> lower=-2.879793 upper=2.879793 effort=1000.0 velocity=0
- joint joint3_to_joint2: limit lower=-2.3562 upper=2.3562 effort=1000.0 velocity=0 -> lower=-2.879793 upper=2.879793 effort=1000.0 velocity=0
- joint joint4_to_joint3: limit lower=-2.618 upper=2.618 effort=1000.0 velocity=0 -> lower=-2.879793 upper=2.879793 effort=1000.0 velocity=0
- joint joint5_to_joint4: limit lower=-2.5307 upper=2.5307 effort=1000.0 velocity=0 -> lower=-2.879793 upper=2.879793 effort=1000.0 velocity=0
- joint joint6_to_joint5: limit lower=-2.8798 upper=2.8798 effort=1000.0 velocity=0 -> lower=-2.879793 upper=2.879793 effort=1000.0 velocity=0
- joint joint6output_to_joint6: limit lower=-3.14159 upper=3.14159 effort=1000.0 velocity=0 -> lower=-3.05 upper=3.05 effort=1000.0 velocity=0

File: mycobot_ros2/mycobot_description/urdf/mycobot_280_m5/mycobot_280_m5_with_pump.urdf (robot description, URDF)
Before this commit: robot firefighter, 10 links, 9 joints
Joints:
- joint joint2_to_joint1: limit lower=-2.9322 upper=2.9322 effort=1000.0 velocity=0 -> lower=-2.879793 upper=2.879793 effort=1000.0 velocity=0
- joint joint3_to_joint2: limit lower=-2.3562 upper=2.3562 effort=1000.0 velocity=0 -> lower=-2.879793 upper=2.879793 effort=1000.0 velocity=0
- joint joint4_to_joint3: limit lower=-2.618 upper=2.618 effort=1000.0 velocity=0 -> lower=-2.879793 upper=2.879793 effort=1000.0 velocity=0
- joint joint5_to_joint4: limit lower=-2.5307 upper=2.5307 effort=1000.0 velocity=0 -> lower=-2.879793 upper=2.879793 effort=1000.0 velocity=0
- joint joint6_to_joint5: limit lower=-2.8798 upper=2.8798 effort=1000.0 velocity=0 -> lower=-2.879793 upper=2.879793 effort=1000.0 velocity=0
- joint joint6output_to_joint6: limit lower=-3.14159 upper=3.14159 effort=1000.0 velocity=0 -> lower=-3.05 upper=3.05 effort=1000.0 velocity=0

File: mycobot_ros2/mycobot_description/urdf/mycobot_280_m5/mycobot_with_vision.urdf (robot description, URDF)
Before this commit: robot mycobot_ai, 8 links, 7 joints
Joints:
- joint joint2_to_joint1: limit lower=-2.9322 upper=2.9322 effort=1000.0 velocity=0 -> lower=-3.14 upper=3.14159 effort=1000.0 velocity=0
- joint joint3_to_joint2: limit lower=-2.3562 upper=2.3562 effort=1000.0 velocity=0 -> lower=-3.14 upper=3.14159 effort=1000.0 velocity=0
- joint joint4_to_joint3: limit lower=-2.618 upper=2.618 effort=1000.0 velocity=0 -> lower=-3.14 upper=3.14159 effort=1000.0 velocity=0
- joint joint5_to_joint4: limit lower=-2.5307 upper=2.5307 effort=1000.0 velocity=0 -> lower=-3.14 upper=3.14159 effort=1000.0 velocity=0
- joint joint6_to_joint5: limit lower=-2.8798 upper=2.8798 effort=1000.0 velocity=0 -> lower=-3.14 upper=3.14159 effort=1000.0 velocity=0
- joint joint6output_to_joint6: limit lower=-3.14159 upper=3.14159 effort=1000.0 velocity=0 -> lower=-3.14 upper=3.14159 effort=1000.0 velocity=0

File: mycobot_ros2/mycobot_description/urdf/mycobot_280_pi/mycobot_280_pi.urdf (robot description, URDF)
Before this commit: robot firefighter, 8 links, 7 joints
Joints:
- joint joint2_to_joint1: limit lower=-2.9322 upper=2.9322 effort=1000.0 velocity=0 -> lower=-3.14 upper=3.14159 effort=1000.0 velocity=0
- joint joint3_to_joint2: limit lower=-2.3562 upper=2.3562 effort=1000.0 velocity=0 -> lower=-3.14 upper=3.14159 effort=1000.0 velocity=0
- joint joint4_to_joint3: limit lower=-2.618 upper=2.618 effort=1000.0 velocity=0 -> lower=-3.14 upper=3.14159 effort=1000.0 velocity=0
- joint joint5_to_joint4: limit lower=-2.5307 upper=2.5307 effort=1000.0 velocity=0 -> lower=-3.14 upper=3.14159 effort=1000.0 velocity=0
- joint joint6_to_joint5: limit lower=-2.8798 upper=2.8798 effort=1000.0 velocity=0 -> lower=-3.14 upper=3.14159 effort=1000.0 velocity=0; origin xyz=0 -0.07318 -0.001 rpy=1.5708 -1.5708 0 -> xyz=0 -0.07318 0 rpy=1.5708 -1.5708 0
- joint joint6output_to_joint6: limit lower=-3.14159 upper=3.14159 effort=1000.0 velocity=0 -> lower=-3.14 upper=3.14159 effort=1000.0 velocity=0

File: mycobot_ros2/mycobot_description/urdf/mycobot_280_pi/mycobot_280_pi_with_camera_flange.urdf (robot description, URDF)
Before this commit: robot firefighter, 9 links, 8 joints
Joints:
- joint joint2_to_joint1: limit lower=-2.9322 upper=2.9322 effort=1000.0 velocity=0 -> lower=-3.14 upper=3.14159 effort=1000.0 velocity=0
- joint joint3_to_joint2: limit lower=-2.3562 upper=2.3562 effort=1000.0 velocity=0 -> lower=-3.14 upper=3.14159 effort=1000.0 velocity=0
- joint joint4_to_joint3: limit lower=-2.618 upper=2.618 effort=1000.0 velocity=0 -> lower=-3.14 upper=3.14159 effort=1000.0 velocity=0
- joint joint5_to_joint4: limit lower=-3.5307 upper=3.5307 effort=1000.0 velocity=0 -> lower=-3.14 upper=3.14159 effort=1000.0 velocity=0
- joint joint6_to_joint5: limit lower=-2.8798 upper=2.8798 effort=1000.0 velocity=0 -> lower=-3.14 upper=3.14159 effort=1000.0 velocity=0; origin xyz=0 -0.07318 -0.001 rpy=1.5708 -1.5708 0 -> xyz=0 -0.07318 0 rpy=1.5708 -1.5708 0
- joint joint6output_to_joint6: limit lower=-3.14159 upper=3.14159 effort=1000.0 velocity=0 -> lower=-3.14 upper=3.14159 effort=1000.0 velocity=0

File: mycobot_ros2/mycobot_description/urdf/mycobot_280_pi/mycobot_280_pi_with_camera_flange_pump.urdf (robot description, URDF)
Before this commit: robot firefighter, 11 links, 10 joints
Joints:
- joint joint2_to_joint1: limit lower=-2.9322 upper=2.9322 effort=1000.0 velocity=0 -> lower=-3.14 upper=3.14159 effort=1000.0 velocity=0
- joint joint3_to_joint2: limit lower=-2.3562 upper=2.3562 effort=1000.0 velocity=0 -> lower=-3.14 upper=3.14159 effort=1000.0 velocity=0
- joint joint4_to_joint3: limit lower=-2.618 upper=2.618 effort=1000.0 velocity=0 -> lower=-3.14 upper=3.14159 effort=1000.0 velocity=0
- joint joint5_to_joint4: limit lower=-2.5307 upper=2.5307 effort=1000.0 velocity=0 -> lower=-3.14 upper=3.14159 effort=1000.0 velocity=0
- joint joint6_to_joint5: limit lower=-2.8798 upper=2.8798 effort=1000.0 velocity=0 -> lower=-3.14 upper=3.14159 effort=1000.0 velocity=0; origin xyz=0 -0.07318 -0.001 rpy=1.5708 -1.5708 0 -> xyz=0 -0.07318 0 rpy=1.5708 -1.5708 0
- joint joint6output_to_joint6: limit lower=-3.14159 upper=3.14159 effort=1000.0 velocity=0 -> lower=-3.14 upper=3.14159 effort=1000.0 velocity=0

File: mycobot_ros2/mycobot_description/urdf/mycobot_280_pi/mycobot_280_pi_with_pump.urdf (robot description, URDF)
Before this commit: robot firefighter, 10 links, 9 joints
Joints:
- joint joint2_to_joint1: limit lower=-2.9322 upper=2.9322 effort=1000.0 velocity=0 -> lower=-3.14 upper=3.14159 effort=1000.0 velocity=0
- joint joint3_to_joint2: limit lower=-2.3562 upper=2.3562 effort=1000.0 velocity=0 -> lower=-3.14 upper=3.14159 effort=1000.0 velocity=0
- joint joint4_to_joint3: limit lower=-2.618 upper=2.618 effort=1000.0 velocity=0 -> lower=-3.14 upper=3.14159 effort=1000.0 velocity=0
- joint joint5_to_joint4: limit lower=-2.5307 upper=2.5307 effort=1000.0 velocity=0 -> lower=-3.14 upper=3.14159 effort=1000.0 velocity=0
- joint joint6_to_joint5: limit lower=-2.8798 upper=2.8798 effort=1000.0 velocity=0 -> lower=-3.14 upper=3.14159 effort=1000.0 velocity=0; origin xyz=0 -0.07318 -0.001 rpy=1.5708 -1.5708 0 -> xyz=0 -0.07318 0 rpy=1.5708 -1.5708 0
- joint joint6output_to_joint6: limit lower=-3.14159 upper=3.14159 effort=1000.0 velocity=0 -> lower=-3.14 upper=3.14159 effort=1000.0 velocity=0

File: mycobot_ros2/mycobot_description/urdf/mycobot_280_x3pi/mycobot_280_x3pi.urdf (robot description, URDF)
Before this commit: robot firefighter, 7 links, 6 joints
Joints:
- joint joint2_to_joint1: limit lower=-2.9322 upper=2.9322 effort=1000.0 velocity=0 -> lower=-3.14 upper=3.14159 effort=1000.0 velocity=0
- joint joint3_to_joint2: limit lower=-2.3562 upper=2.3562 effort=1000.0 velocity=0 -> lower=-3.14 upper=3.14159 effort=1000.0 velocity=0
- joint joint4_to_joint3: limit lower=-2.618 upper=2.618 effort=1000.0 velocity=0 -> lower=-3.14 upper=3.14159 effort=1000.0 velocity=0
- joint joint5_to_joint4: limit lower=-2.5307 upper=2.5307 effort=1000.0 velocity=0 -> lower=-3.14 upper=3.14159 effort=1000.0 velocity=0
- joint joint6_to_joint5: limit lower=-2.8798 upper=2.8798 effort=1000.0 velocity=0 -> lower=-3.14 upper=3.14159 effort=1000.0 velocity=0
- joint joint6output_to_joint6: limit lower=-3.14159 upper=3.14159 effort=1000.0 velocity=0 -> lower=-3.14 upper=3.14159 effort=1000.0 velocity=0

File: mycobot_ros2/mycobot_description/urdf/mycobot_320_m5_2022/mycobot_320_m5_2022.urdf (robot description, URDF)
Before this commit: robot firefighter, 7 links, 6 joints
Joints:
- joint joint2_to_joint1: limit lower=-2.9321 upper=2.9321 effort=1000.0 velocity=0 -> lower=-2.87 upper=2.87 effort=1000.0 velocity=0
- joint joint3_to_joint2: limit lower=-2.3561 upper=2.3561 effort=1000.0 velocity=0 -> lower=-2.879 upper=2.879 effort=1000.0 velocity=0
- joint joint4_to_joint3: limit lower=-2.5307 upper=2.5307 effort=1000.0 velocity=0 -> lower=-2.879 upper=2.879 effort=1000.0 velocity=0
- joint joint5_to_joint4: limit lower=-2.5830 upper=2.5830 effort=1000.0 velocity=0 -> lower=-2.879 upper=2.879 effort=1000.0 velocity=0
- joint joint6_to_joint5: limit lower=-2.9321 upper=2.9321 effort=1000.0 velocity=0 -> lower=-2.879 upper=2.879 effort=1000.0 velocity=0
- joint joint6output_to_joint6: limit lower=-3.14159 upper=3.14159 effort=1000.0 velocity=0 -> lower=-3.05 upper=3.05 effort=1000.0 velocity=0

File: mycobot_ros2/mycobot_description/urdf/mycobot_320_pi_2022/mycobot_320_pi_2022.urdf (robot description, URDF)
Before this commit: robot firefighter, 7 links, 6 joints
Joints:
- joint joint2_to_joint1: limit lower=-2.9321 upper=2.9321 effort=1000.0 velocity=0 -> lower=-2.96 upper=2.96 effort=1000.0 velocity=0
- joint joint3_to_joint2: limit lower=-2.3561 upper=2.3561 effort=1000.0 velocity=0 -> lower=-2.79 upper=2.79 effort=1000.0 velocity=0
- joint joint4_to_joint3: limit lower=-2.5307 upper=2.5307 effort=1000.0 velocity=0 -> lower=-2.79 upper=2.79 effort=1000.0 velocity=0
- joint joint5_to_joint4: limit lower=-2.5830 upper=2.5830 effort=1000.0 velocity=0 -> lower=-2.79 upper=2.79 effort=1000.0 velocity=0
- joint joint6_to_joint5: limit lower=-2.9321 upper=2.9321 effort=1000.0 velocity=0 -> lower=-2.96 upper=2.96 effort=1000.0 velocity=0
- joint joint6output_to_joint6: limit lower=-3.14159 upper=3.14159 effort=1000.0 velocity=0 -> lower=-3.05 upper=3.05 effort=1000.0 velocity=0

File: mycobot_ros2/mycobot_description/urdf/mycobot_pro_600/mycobot_pro_600.urdf (robot description, URDF)
Before this commit: robot firefighter, 7 links, 6 joints
Joints:
- joint joint3_to_joint2: limit lower=-3.14159 upper=3.14159 effort=1000.0 velocity=0 -> lower=-4.7123 upper=1.5708 effort=1000.0 velocity=0; origin xyz=0 0  0 rpy=1.5708 -1.5708 0 -> xyz=0 0  0 rpy=1.5708 0 0
- joint joint5_to_joint4: limit lower=-2.9670 upper=2.9670 effort=1000.0 velocity=0 -> lower=-4.5378 upper=1.3962 effort=1000.0 velocity=0; origin xyz=0.25 0  -0.1091 rpy=0 0 1.5708 -> xyz=0.25 0  -0.1091 rpy=0 0 0

File: mycobot_ros2/mycobot_description/urdf/mycobot_pro_630/mycobot_pro_630.urdf (robot description, URDF)
Before this commit: robot firefighter, 7 links, 6 joints
Joints:
- joint joint2_to_joint1: limit lower=-3.14159 upper=3.14159 effort=1000.0 velocity=0 -> lower=-4.71 upper=1.5707 effort=1000.0 velocity=0; origin xyz=0 0  0 rpy=1.5707 -1.5708 0 -> xyz=0 0  0 rpy=1.5707 0 0
- joint joint4_to_joint3: limit lower=-2.9670 upper=2.9670 effort=1000.0 velocity=0 -> lower=-4.53 upper=1.3962 effort=1000.0 velocity=0; origin xyz=0.267 0  -0.0745 rpy=0 0 1.5708 -> xyz=0.267 0  -0.0745 rpy=0 0 0

File: mycobot_ros2/mycobot_description/urdf/mypalletizer_260_m5/mypalletizer_260_m5.urdf (robot description, URDF)
Before this commit: robot firefighter, 6 links, 5 joints
Links:
- link base: geometry collision mesh filename=package://mycobot_description/urdf/mypallertizer_260_m5/bas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; visual mesh filename=package://mycobot_description/urdf/mypallertizer_260_m5/bas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
- link link1: geometry collision mesh filename=package://mycobot_description/urdf/mypallertizer_260_m5/lin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; visual mesh filename=package://mycobot_description/urdf/mypallertizer_260_m5/lin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
- link link2: geometry collision mesh filename=package://mycobot_description/urdf/mypallertizer_260_m5/lin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; visual mesh filename=package://mycobot_description/urdf/mypallertizer_260_m5/lin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
- link link3: geometry collision mesh filename=package://mycobot_description/urdf/mypallertizer_260_m5/lin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; visual mesh filename=package://mycobot_description/urdf/mypallertizer_260_m5/lin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
- link link4: geometry collision mesh filename=package://mycobot_description/urdf/mypallertizer_260_m5/lin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; visual mesh filename=package://mycobot_description/urdf/mypallertizer_260_m5/lin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
Joints:
- joint joint2_to_joint1: limit lower=-0.0349 upper=1.5708 effort=1000.0 velocity=0 -> lower=-0.014 upper=1.49 effort=1000.0 velocity=0
- joint joint3_to_joint2: limit lower=-1.6057 upper=1.0471 effort=1000.0 velocity=0 -> lower=-0.213 upper=0.872665 effort=1000.0 velocity=0
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